Commit message: hotfix robot description for realRobot

File: description/camera.xacro (robot description, xacro)
@@ -4,5 +4,5 @@
         <parent link="chassis"/>
         <child link="camera_link"/>
-        <origin xyz="0.276 0 0.181" rpy="0 0 0"/>
+        <origin xyz="0.456 0 0.181" rpy="0 0 0"/>
     </joint>
     <link name="camera_link">

File: description/lidar.xacro (robot description, xacro)
@@ -4,10 +4,11 @@
         <parent link="chassis"/>
         <child link="laser_frame"/>
-        <origin xyz="0.122 0 0.212" rpy="0 0 0"/>
+        <origin xyz="0.35 0 0.22" rpy="0 0 0"/>
     </joint>
     <link name="laser_frame">
         <visual>
             <geometry>
-                <cylinder radius="0.05" length="0.04"/>
+                <!-- <cylinder radius="0.035" length="0.025"/> -->
+                 <cylinder radius="0.05" length="0.055"/>
             </geometry>
             <material name="black"/>
@@ -22,8 +23,8 @@
         <collision>
             <geometry>
-                <cylinder radius="0.05" length="0.04"/>
+                <cylinder radius="0.05" length="0.055"/>
             </geometry>
         </collision>
-        <xacro:inertial_cylinder mass="0.1" length="0.04" radius="0.05">
+        <xacro:inertial_cylinder mass="0.2" length="0.055" radius="0.05">
             <origin xyz="0 0 0" rpy="0 0 0"/>
         </xacro:inertial_cylinder>

File: description/robot_core.xacro (robot description, xacro)
@@ -1,21 +1,52 @@
 <?xml version="1.0"?>
-<robot xmlns:xacro="http://www.ros.org/wiki/xacro" >
+<robot xmlns:xacro="http://www.ros.org/wiki/xacro">
     <xacro:include filename="inertial_macros.xacro"/>
-    <xacro:property name="chassis_length" value="0.335"/>
-    <xacro:property name="chassis_width" value="0.265"/>
-    <xacro:property name="chassis_height" value="0.138"/>
-    <xacro:property name="chassis_mass" value="1.0"/>
-    <xacro:property name="wheel_radius" value="0.034"/>
-    <xacro:property name="wheel_thickness" value="0.026"/>
-    <xacro:property name="wheel_mass" value="0.05"/>
-    <xacro:property name="wheel_offset_x" value="0.226"/>
-    <xacro:property name="wheel_offset_y" value="0.166"/>
-    <xacro:property name="wheel_offset_z" value="0.01"/>
-    <xacro:property name="caster_wheel_radius" value="0.01"/>
-    <xacro:property name="caster_wheel_mass" value="0.01"/>
-    <xacro:property name="caster_wheel_offset_x" value="0.075"/>
-    <xacro:property name="caster_wheel_offset_z" value="${wheel_offset_z - wheel_radius + caster_wheel_radius}"/>
+    <!-- ========================================================= -->
+    <!-- ROBOT PARAMETERS                                          -->
+    <!-- ========================================================= -->
+    <xacro:property name="chassis_length" value="0.50"/>
+    <xacro:property name="chassis_width" value="0.40"/>
+    <xacro:property name="chassis_height" value="0.15"/>
+    <xacro:property name="chassis_mass" value="2.50"/>
+    <!-- ========================================================= -->
+    <!-- DRIVE WHEEL PARAMETERS                                    -->
+    <!-- ========================================================= -->
+    <xacro:property name="wheel_radius" value="0.05"/>
+    <xacro:property name="wheel_thickness" value="0.03"/>
+    <xacro:property name="wheel_mass" value="0.18"/>
+    <xacro:property name="wheel_separation" value="0.50"/>
+    <xacro:property name="chassis_offset_x"
+                    value="${chassis_length / 2.0}"/>
+    <xacro:property name="wheel_offset_y"
+                    value="${wheel_separation / 2.0}"/>
+    <xacro:property name="wheel_offset_z"
+                    value="${wheel_radius}"/>
+    <!-- ========================================================= -->
+    <!-- CHASSIS PARAMETERS                                        -->
+    <!-- ========================================================= -->
+    <xacro:property name="ground_clearance"
+                    value="0.025"/>
+    <xacro:property name="chassis_offset_z"
+                    value="${ground_clearance - wheel_offset_z}"/>
+    <!-- ========================================================= -->
+    <!-- CASTER PARAMETERS                                         -->
+    <!-- ========================================================= -->
+    <xacro:property name="caster_wheel_radius"
+                    value="0.010"/>
+    <xacro:property name="caster_wheel_thickness"
+                    value="0.025"/>
+    <xacro:property name="caster_wheel_mass"
+                    value="0.05"/>
+    <xacro:property name="caster_offset_x"
+                    value="0.10"/>
+    <xacro:property name="caster_offset_y"
+                    value="0.15"/>
+    <xacro:property name="caster_offset_z"
+                    value="-0.015"/>
+    <!-- ========================================================= -->
+    <!-- MATERIALS                                                 -->
+    <!-- ========================================================= -->
     <material name="white">
-        <color rgba="1 1 1 1" />
+        <color rgba="1 1 1 1"/>
     </material>
     <material name="orange">
@@ -31,37 +62,71 @@
         <color rgba="1 0 0 1"/>
     </material>
-    <!-- BASE LINK -->
+    <!-- ========================================================= -->
+    <!-- BASE LINK                                                  -->
+    <!-- ========================================================= -->
     <link name="base_link">
     </link>
-    <!-- BASE_FOOTPRINT LINK -->
-     <joint name="base_footprint_joint" type="fixed">
+    <!-- ========================================================= -->
+    <!-- BASE FOOTPRINT                                             -->
+    <!-- ========================================================= -->
+    <joint name="base_footprint_joint" type="fixed">
         <parent link="base_link"/>
         <child link="base_footprint"/>
-        <origin xyz="0 0 0 " rpy="0 0 0"/>
-     </joint>
-     <link name="base_footprint">
-     </link>
-    <!-- CHASSIS LINK -->
+        <origin
+            xyz="0 0 ${-wheel_offset_z}"
+            rpy="0 0 0"/>
+    </joint>
+    <link name="base_footprint">
+    </link>
+    <!-- ========================================================= -->
+    <!-- CHASSIS                                                    -->
+    <!-- ========================================================= -->
     <joint name="chassis_joint" type="fixed">
         <parent link="base_link"/>
         <child link="chassis"/>
-        <origin xyz="${-wheel_offset_x} 0 ${-wheel_offset_z}"/>
+        <origin
+            xyz="${-chassis_offset_x}
+                 0
+                 ${chassis_offset_z}"
+            rpy="0 0 0"/>
     </joint>
     <link name="chassis">
         <visual>
-            <origin xyz="${chassis_length/2} 0 ${chassis_height/2}"/>
-            <geometry>
-                <box size="${chassis_length} ${chassis_width} ${chassis_height}"/>
+            <origin
+                xyz="${chassis_length / 2.0}
+                     0
+                     ${chassis_height / 2.0}"
+                rpy="0 0 0"/>
+            <geometry>
+                <box
+                    size="${chassis_length}
+                          ${chassis_width}
+                          ${chassis_height}"/>
             </geometry>
             <material name="orange"/>
         </visual>
         <collision>
-            <origin xyz="${chassis_length/2} 0 ${chassis_height/2}"/>
-            <geometry>
-                <box size="${chassis_length} ${chassis_width} ${chassis_height}"/>
+            <origin
+                xyz="${chassis_length / 2.0}
+                     0
+                     ${chassis_height / 2.0}"
+                rpy="0 0 0"/>
+            <geometry>
+                <box
+                    size="${chassis_length}
+                          ${chassis_width}
+                          ${chassis_height}"/>
             </geometry>
         </collision>
-        <xacro:inertial_box mass="0.5" x="${chassis_length}" y="${chassis_width}" z="${chassis_height}">
-            <origin xyz="${chassis_length/2} 0 ${chassis_height/2}" rpy="0 0 0"/>
+        <xacro:inertial_box
+            mass="${chassis_mass}"
+            x="${chassis_length}"
+            y="${chassis_width}"
+            z="${chassis_height}">
+            <origin
+                xyz="${chassis_length / 2.0}
+                     0
+                     ${chassis_height / 2.0}"
+                rpy="0 0 0"/>
         </xacro:inertial_box>
     </link>
@@ -69,9 +134,13 @@
         <material>Gazebo/Orange</material>
     </gazebo>
-    <!-- LEFT WHEEL LINK -->
+    <!-- ========================================================= -->
+    <!-- LEFT DRIVE WHEEL                                          -->
+    <!-- ========================================================= -->
     <joint name="left_wheel_joint" type="continuous">
         <parent link="base_link"/>
         <child link="left_wheel"/>
-        <origin xyz="0 ${wheel_offset_y} 0" rpy="-${pi/2} 0 0" />
+        <origin
+            xyz="0 ${wheel_offset_y} 0"
+            rpy="-${pi / 2.0} 0 0"/>
         <axis xyz="0 0 1"/>
     </joint>
@@ -79,5 +148,7 @@
         <visual>
             <geometry>
-                <cylinder radius="${wheel_radius}" length="${wheel_thickness}"/>
+                <cylinder
+                    radius="${wheel_radius}"
+                    length="${wheel_thickness}"/>
             </geometry>
             <material name="blue"/>
@@ -85,19 +156,33 @@
         <collision>
             <geometry>
-                <sphere radius="${wheel_radius}"/>
+                <sphere
+                    radius="${wheel_radius}"/>
             </geometry>
         </collision>
-        <xacro:inertial_cylinder mass="${wheel_mass}" length="${wheel_thickness}" radius="${wheel_radius}">
-            <origin xyz="0 0 0" rpy="0 0 0"/>
+        <xacro:inertial_cylinder
+            mass="${wheel_mass}"
+            length="${wheel_thickness}"
+            radius="${wheel_radius}">
+            <origin
+                xyz="0 0 0"
+                rpy="0 0 0"/>
         </xacro:inertial_cylinder>
     </link>
     <gazebo reference="left_wheel">
         <material>Gazebo/Blue</material>
+        <!-- <mu1 value="1.0"/>
+        <mu2 value="1.0"/> -->
+        <mu1 value="0.7"/>
+        <mu2 value="0.7"/>
     </gazebo>
-    <!-- RIGHT WHEEL LINK -->
+    <!-- ========================================================= -->
+    <!-- RIGHT DRIVE WHEEL                                         -->
+    <!-- ========================================================= -->
     <joint name="right_wheel_joint" type="continuous">
         <parent link="base_link"/>
         <child link="right_wheel"/>
-        <origin xyz="0 ${-wheel_offset_y} 0" rpy="${pi/2} 0 0" />
+        <origin
+            xyz="0 ${-wheel_offset_y} 0"
+            rpy="${pi / 2.0} 0 0"/>
         <axis xyz="0 0 -1"/>
     </joint>
@@ -105,5 +190,7 @@
         <visual>
             <geometry>
-                <cylinder radius="${wheel_radius}" length="${wheel_thickness}"/>
+                <cylinder
+                    radius="${wheel_radius}"
+                    length="${wheel_thickness}"/>
             </geometry>
             <material name="blue"/>
@@ -111,40 +198,85 @@
         <collision>
             <geometry>
-                <sphere radius="${wheel_radius}"/>
+                <sphere
+                    radius="${wheel_radius}"/>
             </geometry>
         </collision>
-        <xacro:inertial_cylinder mass="${wheel_mass}" length="${wheel_thickness}" radius="${wheel_radius}">
-            <origin xyz="0 0 0" rpy="0 0 0"/>
+        <xacro:inertial_cylinder
+            mass="${wheel_mass}"
+            length="${wheel_thickness}"
+            radius="${wheel_radius}">
+            <origin
+                xyz="0 0 0"
+                rpy="0 0 0"/>
         </xacro:inertial_cylinder>
     </link>
     <gazebo reference="right_wheel">
         <material>Gazebo/Blue</material>
+        <mu1 value="1.0"/>
+        <mu2 value="1.0"/>
     </gazebo>
-    <!-- CASTER WHEEL LINK -->
-    <joint name="caster_wheel_joint" type="fixed">
-        <parent link="chassis"/>
-        <child link="caster_wheel"/>
-        <origin xyz="${caster_wheel_offset_x} 0 ${caster_wheel_offset_z}"/>
-    </joint>
-    <link name="caster_wheel">
-        <visual>
-            <geometry>
-                <sphere radius="${caster_wheel_radius}"/>
-            </geometry>
-            <material name="white"/>
-        </visual>
-        <collision>
-            <geometry>
-                <sphere radius="${caster_wheel_radius}"/>
-            </geometry>
-        </collision>
-        <xacro:inertial_sphere mass="${caster_wheel_mass}" radius="${caster_wheel_radius}">
-            <origin xyz="0 0 0" rpy="0 0 0"/>
-        </xacro:inertial_sphere>
-    </link>
-    <gazebo reference="caster_wheel">
-        <material>Gazebo/White</material>
-        <mu1 value="0.001"/>
-        <mu2 value="0.001"/>
-    </gazebo>
+    <!-- ========================================================= -->
+    <!-- CASTER WHEEL MACRO                                        -->
+    <!-- ========================================================= -->
+    <xacro:macro name="caster_wheel" params="name x y">
+        <joint name="${name}_joint" type="fixed">
+            <parent link="chassis"/>
+            <child link="${name}"/>
+            <origin
+                xyz="${x}
+                     ${y}
+                     ${caster_offset_z}"
+                rpy="0 0 0"/>
+        </joint>
+        <link name="${name}">
+            <visual>
+                <origin
+                    xyz="0 0 0"
+                    rpy="${pi / 2.0} 0 0"/>
+                <geometry>
+                    <cylinder
+                        radius="${caster_wheel_radius}"
+                        length="${caster_wheel_thickness}"/>
+                </geometry>
+                <material name="white"/>
+            </visual>
+            <collision>
+                <geometry>
+                    <sphere
+                        radius="${caster_wheel_radius}"/>
+                </geometry>
+            </collision>
+            <xacro:inertial_sphere
+                mass="${caster_wheel_mass}"
+                radius="${caster_wheel_radius}">
+                <origin
+                    xyz="0 0 0"
+                    rpy="0 0 0"/>
+            </xacro:inertial_sphere>
+        </link>
+        <gazebo reference="${name}">
+            <material>Gazebo/White</material>
+            <mu1 value="0.001"/>
+            <mu2 value="0.001"/>
+        </gazebo>
+    </xacro:macro>
+    <!-- ========================================================= -->
+    <!-- FOUR CASTER WHEELS                                        -->
+    <!-- ========================================================= -->
+    <xacro:caster_wheel
+        name="rear_left_caster"
+        x="${caster_offset_x}"
+        y="${caster_offset_y}"/>
+    <xacro:caster_wheel
+        name="rear_right_caster"
+        x="${caster_offset_x}"
+        y="${-caster_offset_y}"/>
+    <xacro:caster_wheel
+        name="front_left_caster"
+        x="${chassis_length - caster_offset_x}"
+        y="${caster_offset_y}"/>
+    <xacro:caster_wheel
+        name="front_right_caster"
+        x="${chassis_length - caster_offset_x}"
+        y="${-caster_offset_y}"/>
 </robot>

File: description/ros2_control.xacro (robot description, xacro)
@@ -71,7 +71,7 @@
                 <left_joint>left_wheel_joint</left_joint>
                 <right_joint>right_wheel_joint</right_joint>
-                <wheel_separation>0.332</wheel_separation>
-                <wheel_diameter>0.068</wheel_diameter>
-                <max_wheel_torque>20</max_wheel_torque>
+                <wheel_separation>0.5</wheel_separation>
+                <wheel_diameter>0.10</wheel_diameter>
+                <max_wheel_torque>3</max_wheel_torque>
                 <max_wheel_acceleration>10.0</max_wheel_acceleration>
                 <command_topic>cmd_vel</command_topic>
