Commit message: add slam_toolbox

File: description/robot_core.xacro (robot description, xacro)
@@ -34,4 +34,12 @@
     <link name="base_link">
     </link>
+    <!-- BASE_FOOTPRINT LINK -->
+     <joint name="base_footprint_joint" type="fixed">
+        <parent link="base_link"/>
+        <child link="base_footprint"/>
+        <origin xyz="0 0 0 " rpy="0 0 0"/>
+     </joint>
+     <link name="base_footprint">
+     </link>
     <!-- CHASSIS LINK -->
     <joint name="chassis_joint" type="fixed">

Commit message: Fix for real robot

File: description/robot_core.xacro (robot description, xacro)
@@ -8,5 +8,5 @@
     <xacro:property name="chassis_width" value="0.40"/>
     <xacro:property name="chassis_height" value="0.15"/>
-    <xacro:property name="chassis_mass" value="2.50"/>
+    <xacro:property name="chassis_mass" value="4.50"/>
     <!-- ========================================================= -->
     <!-- DRIVE WHEEL PARAMETERS                                    -->
@@ -15,9 +15,9 @@
     <xacro:property name="wheel_thickness" value="0.03"/>
     <xacro:property name="wheel_mass" value="0.18"/>
-    <xacro:property name="wheel_separation" value="0.50"/>
+    <xacro:property name="wheel_separation" value="0.35"/>
     <xacro:property name="chassis_offset_x"
                     value="${chassis_length / 2.0}"/>
     <xacro:property name="wheel_offset_y"
-                    value="${wheel_separation / 2.0}"/>
+                    value="${(wheel_separation + 0.15) / 2.0}"/>
     <xacro:property name="wheel_offset_z"
                     value="${wheel_radius}"/>
@@ -26,5 +26,5 @@
     <!-- ========================================================= -->
     <xacro:property name="ground_clearance"
-                    value="0.025"/>
+                    value="0.02"/>
     <xacro:property name="chassis_offset_z"
                     value="${ground_clearance - wheel_offset_z}"/>
@@ -115,5 +115,5 @@
                 <box
                     size="${chassis_length}
-                          ${chassis_width}
+                          ${chassis_width }
                           ${chassis_height}"/>
             </geometry>
