Commit message: Fixing cofig for ros2_controllers

File: description/ros2_control.xacro (robot description, xacro)
@@ -3,5 +3,5 @@
     <ros2_control name="RealRobot" type="system">
         <hardware>
-            <plugin>diffdrive_amrbot/DiffDriveAmrbot</plugin>
+            <plugin>diffdrive_arduino/DiffDriveArduinoHardware</plugin>
             <param name="left_wheel_name">left_wheel_joint</param>
             <param name="right_wheel_name">right_wheel_joint</param>
@@ -9,21 +9,27 @@
             <param name="device">/dev/ttyUSB0</param>
             <param name="baud_rate">115200</param>
-            <param name="time_out">1000</param>
+            <param name="timeout_ms">1000</param>
             <param name="enc_counts_per_rev">1836</param>
+            <!-- <param name="pid_p">13</param>
+            <param name="pid_d">26</param>
+            <param name="pid_i">0</param>
+            <param name="pid_o">30</param> -->
         </hardware>
-        <joint name="left_wheel_joint">
-            <command_interface name="velocity"/>
-                <param name="min">-10</param>
-                <param name="max">10</param>
-            <state_interface name="velocity"/>
-            <state_interface name="position"/>
-        </joint>
-        <joint name="right_wheel_joint">
-            <command_interface name="velocity"/>
-                <param name="min">-10</param>
-                <param name="max">10</param>
-            <state_interface name="velocity"/>
-            <state_interface name="position"/>
-        </joint>
+    <joint name="left_wheel_joint">
+        <command_interface name="velocity">
+            <param name="min">-10</param>
+            <param name="max">10</param>
+        </command_interface>
+        <state_interface name="position"/>
+        <state_interface name="velocity"/>
+    </joint>
+    <joint name="right_wheel_joint">
+        <command_interface name="velocity">
+            <param name="min">-10</param>
+            <param name="max">10</param>
+        </command_interface>
+        <state_interface name="position"/>
+        <state_interface name="velocity"/>
+    </joint>
     </ros2_control>
     <!-- <ros2_control name="GazeboSystem" type="system">

Commit message: Fix gazebo_controller

File: description/ros2_control.xacro (robot description, xacro)
@@ -1,6 +1,7 @@
 <?xml version="1.0"?>
 <robot xmlns:xacro="http://www.ros.org/wiki/xacro">
-    <ros2_control name="RealRobot" type="system">
-        <hardware>
+    <xacro:unless value="$(arg sim_mode)">
+        <ros2_control name="RealRobot" type="system">
+            <hardware>
             <plugin>diffdrive_arduino/DiffDriveArduinoHardware</plugin>
             <param name="left_wheel_name">left_wheel_joint</param>
@@ -16,43 +17,47 @@
             <param name="pid_o">30</param> -->
         </hardware>
-    <joint name="left_wheel_joint">
-        <command_interface name="velocity">
-            <param name="min">-10</param>
-            <param name="max">10</param>
-        </command_interface>
-        <state_interface name="position"/>
-        <state_interface name="velocity"/>
-    </joint>
-    <joint name="right_wheel_joint">
-        <command_interface name="velocity">
-            <param name="min">-10</param>
-            <param name="max">10</param>
-        </command_interface>
-        <state_interface name="position"/>
-        <state_interface name="velocity"/>
-    </joint>
-    </ros2_control>
-    <!-- <ros2_control name="GazeboSystem" type="system">
-        <hardware>
-            <plugin>gazebo_ros2_control/GazeboSystem</plugin>
-        </hardware>
         <joint name="left_wheel_joint">
-            <command_interface name="velocity"/>
+            <command_interface name="velocity">
                 <param name="min">-10</param>
                 <param name="max">10</param>
+            </command_interface>
+            <state_interface name="position"/>
             <state_interface name="velocity"/>
-            <state_interface name="position"/>
         </joint>
         <joint name="right_wheel_joint">
-            <command_interface name="velocity"/>
+            <command_interface name="velocity">
                 <param name="min">-10</param>
                 <param name="max">10</param>
+            </command_interface>
+            <state_interface name="position"/>
             <state_interface name="velocity"/>
-            <state_interface name="position"/>
         </joint>
-    </ros2_control> -->
+        </ros2_control>
+    </xacro:unless>
+    <xacro:if value="$(arg sim_mode)">
+        <ros2_control name="GazeboSystem" type="system">
+            <hardware>
+                <plugin>gazebo_ros2_control/GazeboSystem</plugin>
+            </hardware>
+            <joint name="left_wheel_joint">
+                <command_interface name="velocity"/>
+                    <param name="min">-10</param>
+                    <param name="max">10</param>
+                <state_interface name="velocity"/>
+                <state_interface name="position"/>
+            </joint>
+            <joint name="right_wheel_joint">
+                <command_interface name="velocity"/>
+                    <param name="min">-10</param>
+                    <param name="max">10</param>
+                <state_interface name="velocity"/>
+                <state_interface name="position"/>
+            </joint>
+        </ros2_control>
+    </xacro:if>
     <gazebo>
-        <plugin name="diff_drive" filename="libgazebo_ros2_control.so">
+        <plugin name="gazebo_ros2_control" filename="libgazebo_ros2_control.so">
             <parameters>$(find my_bot)/config/my_controllers.yaml</parameters>
+            <parameters>$(find my_bot)/config/gaz_ros2_ctl_use_sim.yaml</parameters>
         </plugin>
     </gazebo>

Commit message: Fix urdf have solid file

File: description/ros2_control.xacro (robot description, xacro)
@@ -59,6 +59,8 @@
     <gazebo>
         <plugin name="gazebo_ros2_control" filename="libgazebo_ros2_control.so">
-            <parameters>$(find my_bot)/config/my_controllers.yaml</parameters>
-            <parameters>$(find my_bot)/config/gaz_ros2_ctl_use_sim.yaml</parameters>
+            <!-- <parameters>$(find my_bot)/config/my_controllers.yaml</parameters>
+            <parameters>$(find my_bot)/config/gaz_ros2_ctl_use_sim.yaml</parameters> -->
+            <parameters>(find-pkg-share my_bot)/my_controllers.yaml</parameters>
+            <parameters>(find-pkg-share my_bot)/gaz_ros2_ctl_use_sim.yaml</parameters>
         </plugin>
     </gazebo>

File: mybot_core/urdf/mybot_core.urdf (robot description, URDF)
Before this commit: robot my_bot, 9 links, 8 joints
Links:
- removed link base_link
Joints:
- removed joint chassis_joint
